File: pcb/jiran-ble/jiran-ble.kicad_pcb (KiCad board)
At the start: 2 copper layers, 0 parts

Commit message: A lot of things, bruh
Parts:
- added C1: 10uF, jiran-ble:Capacitor_SMD_0805, F.Cu at (44.9, -38.7)
- added C2: 10uF, jiran-ble:Capacitor_SMD_0805, F.Cu at (45.5, -47.2)
- added C3: 10uF, jiran-ble:Capacitor_SMD_0805, F.Cu at (50.3, -47.2)
- added C4: 10uF, jiran-ble:Capacitor_SMD_0805, F.Cu at (179.4, -20.6)
- added C5: 10uF, jiran-ble:Capacitor_SMD_0805, F.Cu at (174.6, -20.6)
- added C6: 10uF, jiran-ble:Capacitor_SMD_0805, F.Cu at (202.8, -30.7)
- added D1: 1N4148, jiran-ble:Diode_SMD_SOD-123, B.Cu at (48.4, 59.5)
- added D10: 1N4148, jiran-ble:Diode_SMD_SOD-123, B.Cu at (105.6, 64.3)
- added D11: 1N4148, jiran-ble:Diode_SMD_SOD-123, B.Cu at (124.6, 69.1)
- added D12: 1N4148, jiran-ble:Diode_SMD_SOD-123, B.Cu at (143.7, 71.4)
- added D13: 1N4148, jiran-ble:Diode_SMD_SOD-123, B.Cu at (48.4, 97.6)
- added D14: 1N4148, jiran-ble:Diode_SMD_SOD-123, B.Cu at (67.5, 95.2)
- added D15: 1N4148, jiran-ble:Diode_SMD_SOD-123, B.Cu at (86.5, 88.1)
- added D16: 1N4148, jiran-ble:Diode_SMD_SOD-123, B.Cu at (105.6, 83.3)
- added D17: 1N4148, jiran-ble:Diode_SMD_SOD-123, B.Cu at (124.6, 88.1)
- added D18: 1N4148, jiran-ble:Diode_SMD_SOD-123, B.Cu at (143.7, 90.5)
- added D19: 1N4148, jiran-ble:Diode_SMD_SOD-123, B.Cu at (48.4, 116.7)
- added D2: 1N4148, jiran-ble:Diode_SMD_SOD-123, B.Cu at (67.5, 57.1)
- added D20: 1N4148, jiran-ble:Diode_SMD_SOD-123, B.Cu at (67.5, 114.3)
- added D21: 1N4148, jiran-ble:Diode_SMD_SOD-123, B.Cu at (86.5, 107.2)
- added D22: 1N4148, jiran-ble:Diode_SMD_SOD-123, B.Cu at (105.6, 102.4)
- added D23: 1N4148, jiran-ble:Diode_SMD_SOD-123, B.Cu at (124.6, 107.2)
- added D24: 1N4148, jiran-ble:Diode_SMD_SOD-123, B.Cu at (143.7, 109.5)
- added D25: 1N4148, jiran-ble:Diode_SMD_SOD-123, B.Cu at (29.4, 92.9)
- added D26: 1N4148, jiran-ble:Diode_SMD_SOD-123, B.Cu at (124.6, 126.2)
- added D27: 1N4148, jiran-ble:Diode_SMD_SOD-123, B.Cu at (143.7, 128.6)
- added D28: 1N4148, jiran-ble:Diode_SMD_SOD-123, B.Cu at (162.7, 131.0)
- added D29: 1N5819, jiran-ble:Diode_SMD_SOD-123, F.Cu at (-22.1, 13.6)
- added D3: 1N4148, jiran-ble:Diode_SMD_SOD-123, B.Cu at (86.5, 50.0)
- added D30: 1N5819, jiran-ble:Diode_SMD_SOD-123, F.Cu at (163.5, -30.5)
- added D31: 1N4148, jiran-ble:Diode_SMD_SOD-123, B.Cu at (307.2, 59.5)
- added D32: 1N4148, jiran-ble:Diode_SMD_SOD-123, B.Cu at (288.1, 57.1)
- added D33: 1N4148, jiran-ble:Diode_SMD_SOD-123, B.Cu at (269.1, 50.0)
- added D34: 1N4148, jiran-ble:Diode_SMD_SOD-123, B.Cu at (250.0, 45.2)
- added D35: 1N4148, jiran-ble:Diode_SMD_SOD-123, B.Cu at (231.0, 50.0)
- added D36: 1N4148, jiran-ble:Diode_SMD_SOD-123, B.Cu at (211.9, 52.4)
- added D37: 1N4148, jiran-ble:Diode_SMD_SOD-123, B.Cu at (307.2, 78.6)
- added D38: 1N4148, jiran-ble:Diode_SMD_SOD-123, B.Cu at (288.1, 76.2)
- added D39: 1N4148, jiran-ble:Diode_SMD_SOD-123, B.Cu at (269.1, 69.1)
- added D4: 1N4148, jiran-ble:Diode_SMD_SOD-123, B.Cu at (105.6, 45.2)
- added D40: 1N4148, jiran-ble:Diode_SMD_SOD-123, B.Cu at (250.0, 64.3)
- added D41: 1N4148, jiran-ble:Diode_SMD_SOD-123, B.Cu at (231.0, 69.1)
- added D42: 1N4148, jiran-ble:Diode_SMD_SOD-123, B.Cu at (211.9, 71.4)
- added D43: 1N4148, jiran-ble:Diode_SMD_SOD-123, B.Cu at (307.2, 97.6)
- added D44: 1N4148, jiran-ble:Diode_SMD_SOD-123, B.Cu at (288.1, 95.2)
- added D45: 1N4148, jiran-ble:Diode_SMD_SOD-123, B.Cu at (269.1, 88.1)
- added D46: 1N4148, jiran-ble:Diode_SMD_SOD-123, B.Cu at (250.0, 83.3)
- added D47: 1N4148, jiran-ble:Diode_SMD_SOD-123, B.Cu at (231.0, 88.1)
- added D48: 1N4148, jiran-ble:Diode_SMD_SOD-123, B.Cu at (211.9, 90.5)
- added D49: 1N4148, jiran-ble:Diode_SMD_SOD-123, B.Cu at (307.2, 116.7)
- added D5: 1N4148, jiran-ble:Diode_SMD_SOD-123, B.Cu at (124.6, 50.0)
- added D50: 1N4148, jiran-ble:Diode_SMD_SOD-123, B.Cu at (288.1, 114.3)
- added D51: 1N4148, jiran-ble:Diode_SMD_SOD-123, B.Cu at (269.1, 107.2)
- added D52: 1N4148, jiran-ble:Diode_SMD_SOD-123, B.Cu at (250.0, 102.4)
- added D53: 1N4148, jiran-ble:Diode_SMD_SOD-123, B.Cu at (231.0, 107.2)
- added D54: 1N4148, jiran-ble:Diode_SMD_SOD-123, B.Cu at (211.9, 109.5)
- added D55: 1N4148, jiran-ble:Diode_SMD_SOD-123, B.Cu at (326.2, 92.9)
- added D56: 1N4148, jiran-ble:Diode_SMD_SOD-123, B.Cu at (231.0, 126.2)
- added D57: 1N4148, jiran-ble:Diode_SMD_SOD-123, B.Cu at (211.9, 128.6)
- added D58: 1N4148, jiran-ble:Diode_SMD_SOD-123, B.Cu at (192.9, 131.0)
- added D6: 1N4148, jiran-ble:Diode_SMD_SOD-123, B.Cu at (143.7, 52.4)
- added D7: 1N4148, jiran-ble:Diode_SMD_SOD-123, B.Cu at (48.4, 78.6)
- added D8: 1N4148, jiran-ble:Diode_SMD_SOD-123, B.Cu at (67.5, 76.2)
- added D9: 1N4148, jiran-ble:Diode_SMD_SOD-123, B.Cu at (86.5, 69.1)
- added F1: 500mA, jiran-ble:Fuse_SMD_0805, F.Cu at (50.1, -41.2)
- added F2: 500mA, jiran-ble:Fuse_SMD_0805, F.Cu at (202.7, -27.7)
- added G1: logo-jiran-hotswap, jiran-ble:logotype, F.Cu at (-85.0, 22.6)
- added G2: logo-jiran-hotswap, jiran-ble:logotype, F.Cu at (-73.8, 22.6)
- added HM1: CaseHole, used_footprints:Hole_Mount_M4, F.Cu at (54.4, -54.4)
- added HM10: CaseHole, used_footprints:Hole_Mount_M4, F.Cu at (191.5, -22.9)
- added HM2: CaseHole, used_footprints:Hole_Mount_M4, F.Cu at (39.9, -42.8)
- added HM3: CaseHole, used_footprints:Hole_Mount_M4, F.Cu at (45.1, -42.8)
- added HM4: CaseHole, used_footprints:Hole_Mount_M4, F.Cu at (39.9, -37.6)
- added HM5: CaseHole, used_footprints:Hole_Mount_M4, F.Cu at (54.4, -59.6)
- added HM6: CaseHole, used_footprints:Hole_Mount_M4, F.Cu at (275.9, -110.4)
- added HM7: CaseHole, used_footprints:Hole_Mount_M4, F.Cu at (186.3, -22.9)
- added HM8: CaseHole, used_footprints:Hole_Mount_M4, F.Cu at (197.8, -29.6)
- added HM9: CaseHole, used_footprints:Hole_Mount_M4, F.Cu at (275.9, -105.2)
- added J1: Conn_01x02, jiran-ble:Connector_THT_1x2_2.54, F.Cu at (-43.4, 18.4)
- added J2: Conn_01x04, jiran-ble:Connector_THT_1x4_2.54, F.Cu at (-52.7, 10.9)
- added J3: Conn_01x02, jiran-ble:Connector_THT_1x2_2.54, F.Cu at (-38.8, 12.1)
- added J4: Conn_01x02, jiran-ble:Connector_THT_1x2_2.54, F.Cu at (-48.1, 18.4)
- added J5: Conn_01x02, jiran-ble:Connector_THT_1x2_2.54, F.Cu at (131.8, -22.3)
- added J6: Conn_01x04, jiran-ble:Connector_THT_1x4_2.54, F.Cu at (127.1, -29.9)
- added J7: Conn_01x02, jiran-ble:Connector_THT_1x2_2.54, F.Cu at (141.1, -23.6)
- added J8: Conn_01x02, jiran-ble:Connector_THT_1x2_2.54, F.Cu at (136.4, -22.3)
- added LED1: BT, jiran-ble:LED_SMD_0805, F.Cu at (51.2, -50.3)
- added LED2: CHG, jiran-ble:LED_SMD_0805, F.Cu at (50.1, -44.2)
- added LED3: BT, jiran-ble:LED_SMD_0805, F.Cu at (255.5, -76.9)
- added LED4: CHG, jiran-ble:LED_SMD_0805, F.Cu at (207.6, -30.7)
- added Q1: AO3407, jiran-ble:Package_SMD_SOT-23, F.Cu at (44.7, -34.9)
- added Q2: AO3407, jiran-ble:Package_SMD_SOT-23, F.Cu at (275.5, -95.7)
- added R1: 100K, jiran-ble:Resistor_SMD_0805, F.Cu at (56.0, -47.4)
- added R10: 5.1K, jiran-ble:Resistor_SMD_0805, F.Cu at (235.2, -50.9)
- added R11: 5.1K, jiran-ble:Resistor_SMD_0805, F.Cu at (201.2, -20.9)
- added R12: 1K, jiran-ble:Resistor_SMD_0805, F.Cu at (201.3, -24.8)
- added R13: 100K, jiran-ble:Resistor_SMD_0805, F.Cu at (212.3, -30.7)
- added R14: 100K, jiran-ble:Resistor_SMD_0805, F.Cu at (206.0, -24.8)
- added R15: 1K, jiran-ble:Resistor_SMD_0805, F.Cu at (260.2, -77.0)
- added R16: 4.7K, jiran-ble:Resistor_SMD_0805, F.Cu at (255.4, -73.9)
- added R2: 4.7K, jiran-ble:Resistor_SMD_0805, F.Cu at (-11.0, 19.7)
- added R3: 100K, jiran-ble:Resistor_SMD_0805, F.Cu at (-5.33, 13.0)
- added R4: 5.1K, jiran-ble:Resistor_SMD_0805, F.Cu at (19.5, -10.2)
- added R5: 5.1K, jiran-ble:Resistor_SMD_0805, F.Cu at (-5.33, 10.0)
- added R6: 1K, jiran-ble:Resistor_SMD_0805, F.Cu at (-11.1, 16.7)
- added R7: 1K, jiran-ble:Resistor_SMD_0805, F.Cu at (-15.7, 20.1)
- added R8: 10K, jiran-ble:Resistor_SMD_0805, F.Cu at (56.0, -50.3)
- added R9: 10K, jiran-ble:Resistor_SMD_0805, F.Cu at (196.4, -20.9)
- added SW1: SW_Push, jiran-ble:Switch_Mx_Hotswap_1u, F.Cu at (55.6, 55.6)
- added SW10: SW_Push, jiran-ble:Switch_Mx_Hotswap_1u, F.Cu at (112.7, 60.3)
- added SW11: SW_Push, jiran-ble:Switch_Mx_Hotswap_1u, F.Cu at (131.8, 65.1)
- added SW12: SW_Push, jiran-ble:Switch_Mx_Hotswap_1u, F.Cu at (150.8, 67.5)
- added SW13: SW_Push, jiran-ble:Switch_Mx_Hotswap_1u, F.Cu at (55.6, 93.7)
- added SW14: SW_Push, jiran-ble:Switch_Mx_Hotswap_1u, F.Cu at (74.6, 91.3)
- added SW15: SW_Push, jiran-ble:Switch_Mx_Hotswap_1u, F.Cu at (93.7, 84.1)
- added SW16: SW_Push, jiran-ble:Switch_Mx_Hotswap_1u, F.Cu at (112.7, 79.4)
- added SW17: SW_Push, jiran-ble:Switch_Mx_Hotswap_1u, F.Cu at (131.8, 84.1)
- added SW18: SW_Push, jiran-ble:Switch_Mx_Hotswap_1u, F.Cu at (150.8, 86.5)
- added SW19: SW_Push, jiran-ble:Switch_Mx_Hotswap_1u, F.Cu at (55.6, 112.7)
- added SW2: SW_Push, jiran-ble:Switch_Mx_Hotswap_1u, F.Cu at (74.6, 53.2)
- added SW20: SW_Push, jiran-ble:Switch_Mx_Hotswap_1u, F.Cu at (74.6, 110.3)
- added SW21: SW_Push, jiran-ble:Switch_Mx_Hotswap_1u, F.Cu at (93.7, 103.2)
- added SW22: SW_Push, jiran-ble:Switch_Mx_Hotswap_1u, F.Cu at (112.7, 98.4)
- added SW23: SW_Push, jiran-ble:Switch_Mx_Hotswap_1u, F.Cu at (131.8, 103.2)
- added SW24: SW_Push, jiran-ble:Switch_Mx_Hotswap_1u, F.Cu at (150.8, 105.6)
- added SW25: SW_Push, jiran-ble:Switch_Mx_Hotswap_1u, F.Cu at (36.5, 88.9)
- added SW26: SW_Push, jiran-ble:Switch_Mx_Hotswap_1u, F.Cu at (131.8, 122.2)
- added SW27: SW_Push, jiran-ble:Switch_Mx_Hotswap_1u, F.Cu at (150.8, 124.6)
- added SW28: SW_Push, jiran-ble:Switch_Mx_Hotswap_1u, F.Cu at (169.9, 127.0)
- added SW29: MSK-12C02, jiran-ble:Switch_SMD_MSK-12C02, F.Cu at (-45.8, 11.9)
- added SW3: SW_Push, jiran-ble:Switch_Mx_Hotswap_1u, F.Cu at (93.7, 46.0)
- added SW30: SW_PUSH, jiran-ble:Switch_SMD_Tact_3-6-3,5, F.Cu at (-63.6, 19.4)
- added SW31: SW_PUSH, jiran-ble:Switch_SMD_Tact_3-6-3,5, F.Cu at (143.4, -30.2)
- added SW32: MSK-12C02, jiran-ble:Switch_SMD_MSK-12C02, F.Cu at (134.1, -28.8)
- added SW33: SW_Push, jiran-ble:Switch_Mx_Hotswap_1u, F.Cu at (314.3, 55.6)
- added SW34: SW_Push, jiran-ble:Switch_Mx_Hotswap_1u, F.Cu at (295.3, 53.2)
- added SW35: SW_Push, jiran-ble:Switch_Mx_Hotswap_1u, F.Cu at (276.2, 46.0)
- added SW36: SW_Push, jiran-ble:Switch_Mx_Hotswap_1u, F.Cu at (257.2, 41.3)
- added SW37: SW_Push, jiran-ble:Switch_Mx_Hotswap_1u, F.Cu at (238.1, 46.0)
- added SW38: SW_Push, jiran-ble:Switch_Mx_Hotswap_1u, F.Cu at (219.1, 48.4)
- added SW39: SW_Push, jiran-ble:Switch_Mx_Hotswap_1u, F.Cu at (314.3, 74.6)
- added SW4: SW_Push, jiran-ble:Switch_Mx_Hotswap_1u, F.Cu at (112.7, 41.3)
- added SW40: SW_Push, jiran-ble:Switch_Mx_Hotswap_1u, F.Cu at (295.3, 72.2)
- added SW41: SW_Push, jiran-ble:Switch_Mx_Hotswap_1u, F.Cu at (276.2, 65.1)
- added SW42: SW_Push, jiran-ble:Switch_Mx_Hotswap_1u, F.Cu at (257.2, 60.3)
- added SW43: SW_Push, jiran-ble:Switch_Mx_Hotswap_1u, F.Cu at (238.1, 65.1)
- added SW44: SW_Push, jiran-ble:Switch_Mx_Hotswap_1u, F.Cu at (219.1, 67.5)
- added SW45: SW_Push, jiran-ble:Switch_Mx_Hotswap_1u, F.Cu at (314.3, 93.7)
- added SW46: SW_Push, jiran-ble:Switch_Mx_Hotswap_1u, F.Cu at (295.3, 91.3)
- added SW47: SW_Push, jiran-ble:Switch_Mx_Hotswap_1u, F.Cu at (276.2, 84.1)
- added SW48: SW_Push, jiran-ble:Switch_Mx_Hotswap_1u, F.Cu at (257.2, 79.4)
- added SW49: SW_Push, jiran-ble:Switch_Mx_Hotswap_1u, F.Cu at (238.1, 84.1)
- added SW5: SW_Push, jiran-ble:Switch_Mx_Hotswap_1u, F.Cu at (131.8, 46.0)
- added SW50: SW_Push, jiran-ble:Switch_Mx_Hotswap_1u, F.Cu at (219.1, 86.5)
- added SW51: SW_Push, jiran-ble:Switch_Mx_Hotswap_1u, F.Cu at (314.3, 112.7)
- added SW52: SW_Push, jiran-ble:Switch_Mx_Hotswap_1u, F.Cu at (295.3, 110.3)
- added SW53: SW_Push, jiran-ble:Switch_Mx_Hotswap_1u, F.Cu at (276.2, 103.2)
- added SW54: SW_Push, jiran-ble:Switch_Mx_Hotswap_1u, F.Cu at (257.2, 98.4)
- added SW55: SW_Push, jiran-ble:Switch_Mx_Hotswap_1u, F.Cu at (238.1, 103.2)
- added SW56: SW_Push, jiran-ble:Switch_Mx_Hotswap_1u, F.Cu at (219.1, 105.6)
- added SW57: SW_Push, jiran-ble:Switch_Mx_Hotswap_1u, F.Cu at (333.4, 88.9)
- added SW58: SW_Push, jiran-ble:Switch_Mx_Hotswap_1u, F.Cu at (238.1, 122.2)
- added SW59: SW_Push, jiran-ble:Switch_Mx_Hotswap_1u, F.Cu at (219.1, 124.6)
- added SW6: SW_Push, jiran-ble:Switch_Mx_Hotswap_1u, F.Cu at (150.8, 48.4)
- added SW60: SW_Push, jiran-ble:Switch_Mx_Hotswap_1u, F.Cu at (200.0, 127.0)
- added SW7: SW_Push, jiran-ble:Switch_Mx_Hotswap_1u, F.Cu at (55.6, 74.6)
- added SW8: SW_Push, jiran-ble:Switch_Mx_Hotswap_1u, F.Cu at (74.6, 72.2)
- added SW9: SW_Push, jiran-ble:Switch_Mx_Hotswap_1u, F.Cu at (93.7, 65.1)
- added U1: E73-2G4M08S1C, jiran-ble:E73-2G4M08S1C-52840, F.Cu at (-48.4, 66.7)
- added U2: MCP73831, jiran-ble:Package_SMD_SOT-23-5, F.Cu at (39.0, -32.6)
- added U3: AP2112K-3.3, jiran-ble:Package_SMD_SOT-23-5, F.Cu at (13.8, -5.99)
- added U4: USBLC6-2SC6, jiran-ble:Package_SMD_SOT-23-6, F.Cu at (34.0, -26.3)
- added U5: USBLC6-2SC6, jiran-ble:Package_SMD_SOT-23-6, F.Cu at (274.8, -90.5)
- added U6: AP2112K-3.3, jiran-ble:Package_SMD_SOT-23-5, F.Cu at (275.7, -100.3)
- added U7: E73-2G4M08S1C, jiran-ble:E73-2G4M08S1C-52840, F.Cu at (262.7, -85.6)
- added U8: MCP73831, jiran-ble:Package_SMD_SOT-23-5, F.Cu at (196.5, -24.7)
- added USB1: USB_C_Receptacle_USB2.0, jiran-ble:USB-C_MidMount, F.Cu at (-57.1, 35.7)
- added USB2: USB_C_Receptacle_USB2.0, jiran-ble:USB-C_MidMount, F.Cu at (118.2, -28.5)
