File: pcb/jiran-ble/jiran-ble.kicad_pcb (KiCad board)
At the start: 2 copper layers, 178 parts, among them J1 Conn_01x02, J2 Conn_01x04, J3 Conn_01x02, J4 Conn_01x02, J5 Conn_01x02, J6 Conn_01x04, J7 Conn_01x02, J8 Conn_01x02, Q1 AO3407, Q2 AO3407, SW1 SW_Push, SW10 SW_Push, SW11 SW_Push, SW12 SW_Push, SW13 SW_Push, SW14 SW_Push, SW15 SW_Push, SW16 SW_Push, SW17 SW_Push, SW18 SW_Push, SW19 SW_Push, SW2 SW_Push, SW20 SW_Push, SW21 SW_Push, SW22 SW_Push, SW23 SW_Push, SW24 SW_Push, SW25 SW_Push, SW26 SW_Push, SW27 SW_Push, SW28 SW_Push, SW29 MSK-12C02, SW3 SW_Push, SW30 SW_PUSH, SW31 SW_PUSH, SW32 MSK-12C02, SW33 SW_Push, SW34 SW_Push, SW35 SW_Push, SW36 SW_Push, SW37 SW_Push, SW38 SW_Push, SW39 SW_Push, SW4 SW_Push, SW40 SW_Push, SW41 SW_Push, SW42 SW_Push, SW43 SW_Push, SW44 SW_Push, SW45 SW_Push, SW46 SW_Push, SW47 SW_Push, SW48 SW_Push, SW49 SW_Push, SW5 SW_Push, SW50 SW_Push, SW51 SW_Push, SW52 SW_Push, SW53 SW_Push, SW54 SW_Push, SW55 SW_Push, SW56 SW_Push, SW57 SW_Push, SW58 SW_Push, SW59 SW_Push, SW6 SW_Push, SW60 SW_Push, SW7 SW_Push, SW8 SW_Push, SW9 SW_Push, U1 E73-2G4M08S1C, U2 MCP73831, U3 AP2112K-3.3, U4 USBLC6-2SC6, U5 USBLC6-2SC6, U6 AP2112K-3.3, U7 E73-2G4M08S1C, U8 MCP73831

Commit message: I am veeeery lazy...
Parts:
- removed C1, C2, C3, C4, C5, C6: 10uF, jiran-ble:Capacitor_SMD_0805
- removed F1, F2: 500mA, jiran-ble:Fuse_SMD_0805
- removed J7, J8: Conn_01x02, jiran-ble:Connector_THT_1x2_2.54
- removed Q2: AO3407, jiran-ble:Package_SMD_SOT-23
- removed R14: 100K, jiran-ble:Resistor_SMD_0805
- removed R6: 1K, jiran-ble:Resistor_SMD_0805
- removed SW59, SW60: SW_Push, jiran-ble:Switch_Mx_Hotswap_1u
- removed U7: E73-2G4M08S1C, jiran-ble:E73-2G4M08S1C-52840
- removed U8: MCP73831, jiran-ble:Package_SMD_SOT-23-5
- removed USB1, USB2: USB_C_Receptacle_USB2.0, jiran-ble:USB-C_MidMount
- added P1: Breakoff, jiran-ble:Panel_2x5, F.Cu at (174.6, 127.0)
- added P2: Breakoff, jiran-ble:Panel_2x5, F.Cu at (174.6, 49.2)
- added P3: Breakoff, jiran-ble:Panel_2x5, F.Cu at (192.9, 49.2)
- added P4: Breakoff, jiran-ble:Panel_2x5, F.Cu at (192.9, 127.0)
- added Q3: AO3407, jiran-ble:Package_SMD_SOT-23, B.Cu at (204.0, 60.3)
- added R17: 1K, jiran-ble:Resistor_SMD_0805, F.Cu at (208.1, 70.6)
- added R18: RPROG, jiran-ble:Resistor_SMD_0805, F.Cu at (203.4, 70.6)
- added X1: Crystal, jiran-ble:Crystal_SMD_CM9V, B.Cu at (160.2, 57.9)
- added X2: Crystal, jiran-ble:Crystal_SMD_CM9V, B.Cu at (207.4, 64.3)
- D1: value 1N4148 -> 1N5819
- D29: value 1N5819 -> 1N4148; moved to B.Cu
- D30, G1, Q1: moved to B.Cu
- HM1, HM10, HM2, HM3, HM4, HM5, HM6, HM7, HM8, HM9: footprint used_footprints:Hole_Mount_M4 -> jiran-ble:Hole_Mount_M4
- J1, J4: value Conn_01x02 -> BATT
- J2: value Conn_01x04 -> USB-C Conn; footprint jiran-ble:Connector_THT_1x4_2.54 -> jiran-ble:USB-C_MidMount
- J3: value Conn_01x02 -> SWD; footprint jiran-ble:Connector_THT_1x2_2.54 -> jiran-ble:Connector_THT_1x4_2.54
- J5: value Conn_01x02 -> USB-C Conn; footprint jiran-ble:Connector_THT_1x2_2.54 -> jiran-ble:USB-C_MidMount
- J6: value Conn_01x04 -> SWD
- LED2, LED4: value CHG -> RED
- R1: value 100K -> 5.1K
- R12: value 1K -> 820K
- R13, R3: value 100K -> 1K
- R15: value 1K -> 100K
- R16: value 4.7K -> 2M
- R2: value 4.7K -> 5.1K
- R4: value 5.1K -> 100K
- R5: value 5.1K -> 820K
- R7: value 1K -> 2M
- R8: value 10K -> 1K
- R9: value 10K -> RPROG
- SW1: value SW_Push -> SW_PUSH; footprint jiran-ble:Switch_Mx_Hotswap_1u -> jiran-ble:Switch_SMD_Tact_3-6-3,5
- SW29, SW32: value MSK-12C02 -> SW_Push; footprint jiran-ble:Switch_SMD_MSK-12C02 -> jiran-ble:Switch_Mx_Hotswap_1u
- SW31: value SW_PUSH -> SW_Push; footprint jiran-ble:Switch_SMD_Tact_3-6-3,5 -> jiran-ble:Switch_Mx_Hotswap_1u
- U1: value E73-2G4M08S1C -> XC6220B331MR-G; footprint jiran-ble:E73-2G4M08S1C-52840 -> jiran-ble:Package_SMD_SOT-23-5; moved to B.Cu
- U2: value MCP73831 -> E73-2G4M08S1C; footprint jiran-ble:Package_SMD_SOT-23-5 -> jiran-ble:E73-2G4M08S1C-52840
- U3, U6: value AP2112K-3.3 -> TP4054; moved to B.Cu
- U4: value USBLC6-2SC6 -> XC6220B331MR-G; footprint jiran-ble:Package_SMD_SOT-23-6 -> jiran-ble:Package_SMD_SOT-23-5; moved to B.Cu
- U5: value USBLC6-2SC6 -> E73-2G4M08S1C; footprint jiran-ble:Package_SMD_SOT-23-6 -> jiran-ble:E73-2G4M08S1C-52840
- moved G1 271.4 mm to (183.8, 60.3), turned to 180 degrees
- moved SW30 266.2 mm to (196.1, 78.2), turned to 270 degrees
- moved J4 263.1 mm to (207.5, 81.0), turned to 270 degrees
- moved G2 260.3 mm to (183.8, 60.3)
- moved SW29 238.8 mm to (163.5, 127.0), turned to 180 degrees
- moved HM6 228.4 mm to (232.6, 113.9)
- moved J2 219.1 mm to (163.5, 46.0)
- moved D29 213.6 mm to (156.4, 131.0), turned to 270 degrees
- moved J1 212.9 mm to (160.0, 81.0), turned to 90 degrees
- moved HM9 209.8 mm to (308.8, 102.0)
- moved U1 208.0 mm to (159.6, 61.9), turned to 270 degrees
- moved J3 207.9 mm to (158.8, 77.0), turned to 90 degrees
- moved SW31 194.8 mm to (318.3, 55.6), turned to 180 degrees
- moved U4 194.4 mm to (208.0, 60.3), turned to 90 degrees
- moved HM1 186.6 mm to (134.9, 113.9)
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Connections:
- D1 pad 1: /P1.11_l -> Net-(D1-Pad1)
- D1 pad 2: Net-(D1-Pad2) -> VBUS_l
- D13 pad 1: /P1.13_l -> /P0.28_l
- D19 pad 1: /P0.02_l -> /P1.13_l
- D25 pad 1: /P0.29_l -> /P0.02_l
- D29 pad 1: Net-(C3-Pad1) -> /P0.29_l
- D29 pad 2: VBUS_l -> Net-(D29-Pad2)
- D30 pad 1: Net-(C4-Pad1) -> Net-(D30-Pad1)
- D7 pad 1: /P0.28_l -> /P1.11_l
- J3 pad 2: VBAT_l -> nRF_VDD_l
- J4 pad 2: VBUS_l -> VBAT_r
- J6 pad 2: VCC -> nRF_VDD_r
- Q1 pad 2: Net-(C3-Pad1) -> Net-(D1-Pad1)
- Q1 pad 3: Net-(Q1-Pad3) -> VBAT_l
- R1 pad 1: Net-(C3-Pad1) -> Net-(J2-PadA5)
- R1 pad 2: Net-(R1-Pad2) -> GND
- R10 pad 1: GND -> Net-(J5-PadA5)
- R10 pad 2: Net-(R10-Pad2) -> GND
- R11 pad 1: GND -> Net-(J5-PadB5)
- R11 pad 2: Net-(R11-Pad2) -> GND
- R12 pad 1: Net-(LED3-Pad1) -> VBAT_r
- R12 pad 2: GND -> BATTERY_PIN_r
- R13 pad 1: Net-(C4-Pad1) -> Net-(LED3-Pad1)
- R13 pad 2: Net-(R13-Pad2) -> GND
- R15 pad 1: Net-(LED4-Pad1) -> VBUS_r
- R15 pad 2: Net-(R15-Pad2) -> GND
- R16 pad 1: Net-(R16-Pad1) -> BATTERY_PIN_r
- R2 pad 1: Net-(R2-Pad1) -> Net-(J2-PadB5)
- R3 pad 1: VBUS_l -> Net-(LED1-Pad1)
- R4 pad 1: GND -> VBUS_l
- R4 pad 2: Net-(R4-Pad2) -> GND
- R5 pad 1: GND -> VBAT_l
- R5 pad 2: Net-(R5-Pad2) -> BATTERY_PIN_l
- R7 pad 1: Net-(LED2-Pad1) -> BATTERY_PIN_l
- R7 pad 2: Net-(R7-Pad2) -> GND
- R8 pad 1: Net-(Q1-Pad3) -> Net-(LED2-Pad1)
- R8 pad 2: P0.04_l -> Net-(R8-Pad2)
- R9 pad 1: Net-(Q2-Pad3) -> Net-(R9-Pad1)
- R9 pad 2: P0.04_r -> GND
- SW1 pad 1: Net-(D1-Pad2) -> RESET_l
- SW1 pad 2: /P0.31_l -> GND
- SW10 pad 2: /P0.08_l -> /P0.06_l
- SW11 pad 2: /P0.09_l -> /P0.08_l
- SW12 pad 2: /P0.12_l -> /P0.09_l
- SW13 pad 2: /P0.31_l -> /P0.12_l
- SW14 pad 2: /P0.30_l -> /P0.31_l
- SW15 pad 2: /P0.06_l -> /P0.30_l
- SW16 pad 2: /P0.08_l -> /P0.06_l
- SW17 pad 2: /P0.09_l -> /P0.08_l
- SW18 pad 2: /P0.12_l -> /P0.09_l
- SW19 pad 2: /P0.31_l -> /P0.12_l
- SW2 pad 2: /P0.30_l -> /P0.31_l
- SW20 pad 2: /P0.30_l -> /P0.31_l
- SW21 pad 2: /P0.06_l -> /P0.30_l
- SW22 pad 2: /P0.08_l -> /P0.06_l
- SW23 pad 2: /P0.09_l -> /P0.08_l
- SW24 pad 2: /P0.12_l -> /P0.09_l
- SW25 pad 2: /P0.31_l -> /P0.12_l
- SW26 pad 2: /P0.08_l -> /P0.31_l
- SW27 pad 2: /P0.09_l -> /P0.08_l
- SW28 pad 2: /P0.12_l -> /P0.09_l
- SW29 pad 1: Net-(SW29-Pad1) -> Net-(D29-Pad2)
- SW29 pad 2: VBAT_l -> /P0.12_l
- SW3 pad 2: /P0.06_l -> /P0.30_l
- SW30 pad 1: RESET_l -> RESET_r
- SW31 pad 1: RESET_r -> Net-(D31-Pad2)
- SW31 pad 2: GND -> /P0.31_r
- SW32 pad 1: Net-(SW32-Pad1) -> Net-(D32-Pad2)
- SW32 pad 2: VBAT_r -> /P0.30_r
- SW33 pad 1: Net-(D31-Pad2) -> Net-(D33-Pad2)
- SW33 pad 2: /P0.31_r -> /P0.06_r
- SW34 pad 1: Net-(D32-Pad2) -> Net-(D34-Pad2)
- SW34 pad 2: /P0.30_r -> /P0.08_r
- SW35 pad 1: Net-(D33-Pad2) -> Net-(D35-Pad2)
- SW35 pad 2: /P0.06_r -> /P0.09_r
- SW36 pad 1: Net-(D34-Pad2) -> Net-(D36-Pad2)
- SW36 pad 2: /P0.08_r -> /P0.12_r
- SW37 pad 1: Net-(D35-Pad2) -> Net-(D37-Pad2)
- SW37 pad 2: /P0.09_r -> /P0.31_r
- SW38 pad 1: Net-(D36-Pad2) -> Net-(D38-Pad2)
- SW38 pad 2: /P0.12_r -> /P0.30_r
- SW39 pad 1: Net-(D37-Pad2) -> Net-(D39-Pad2)
- SW39 pad 2: /P0.31_r -> /P0.06_r
- SW4 pad 2: /P0.08_l -> /P0.06_l
- SW40 pad 1: Net-(D38-Pad2) -> Net-(D40-Pad2)
- SW40 pad 2: /P0.30_r -> /P0.08_r
- SW41 pad 1: Net-(D39-Pad2) -> Net-(D41-Pad2)
- SW41 pad 2: /P0.06_r -> /P0.09_r
- SW42 pad 1: Net-(D40-Pad2) -> Net-(D42-Pad2)
- SW42 pad 2: /P0.08_r -> /P0.12_r
- SW43 pad 1: Net-(D41-Pad2) -> Net-(D43-Pad2)
- SW43 pad 2: /P0.09_r -> /P0.31_r
- SW44 pad 1: Net-(D42-Pad2) -> Net-(D44-Pad2)
- SW44 pad 2: /P0.12_r -> /P0.30_r
- SW45 pad 1: Net-(D43-Pad2) -> Net-(D45-Pad2)
- SW45 pad 2: /P0.31_r -> /P0.06_r
- SW46 pad 1: Net-(D44-Pad2) -> Net-(D46-Pad2)
- SW46 pad 2: /P0.30_r -> /P0.08_r
- SW47 pad 1: Net-(D45-Pad2) -> Net-(D47-Pad2)
- SW47 pad 2: /P0.06_r -> /P0.09_r
- SW48 pad 1: Net-(D46-Pad2) -> Net-(D48-Pad2)
- SW48 pad 2: /P0.08_r -> /P0.12_r
- SW49 pad 1: Net-(D47-Pad2) -> Net-(D49-Pad2)
- SW49 pad 2: /P0.09_r -> /P0.31_r
- SW5 pad 2: /P0.09_l -> /P0.08_l
- SW50 pad 1: Net-(D48-Pad2) -> Net-(D50-Pad2)
- SW50 pad 2: /P0.12_r -> /P0.30_r
- SW51 pad 1: Net-(D49-Pad2) -> Net-(D51-Pad2)
- SW51 pad 2: /P0.31_r -> /P0.06_r
- SW52 pad 1: Net-(D50-Pad2) -> Net-(D52-Pad2)
- SW52 pad 2: /P0.30_r -> /P0.08_r
- SW53 pad 1: Net-(D51-Pad2) -> Net-(D53-Pad2)
- SW53 pad 2: /P0.06_r -> /P0.09_r
- SW54 pad 1: Net-(D52-Pad2) -> Net-(D54-Pad2)
- SW54 pad 2: /P0.08_r -> /P0.12_r
- SW55 pad 1: Net-(D53-Pad2) -> Net-(D55-Pad2)
- SW55 pad 2: /P0.09_r -> /P0.31_r
- SW56 pad 1: Net-(D54-Pad2) -> Net-(D56-Pad2)
- SW56 pad 2: /P0.12_r -> /P0.08_r
- SW57 pad 1: Net-(D55-Pad2) -> Net-(D57-Pad2)
- SW57 pad 2: /P0.31_r -> /P0.09_r
- SW58 pad 1: Net-(D56-Pad2) -> Net-(D58-Pad2)
- SW58 pad 2: /P0.08_r -> /P0.12_r
- SW6 pad 2: /P0.12_l -> /P0.09_l
- SW7 pad 2: /P0.31_l -> /P0.12_l
- SW8 pad 2: /P0.30_l -> /P0.31_l
- SW9 pad 2: /P0.06_l -> /P0.30_l
- U1 pad 1: /P1.11_l -> Net-(D1-Pad1)
- U1 pad 2: BLUE_LED_l -> GND
- U1 pad 3: Net-(U1-Pad3) -> Net-(D1-Pad1)
- U1 pad 4: /P0.28_l -> (no net)
- U1 pad 5: GND -> nRF_VDD_l
- U2 pad 1: Net-(R7-Pad2) -> /P1.11_l
- U2 pad 2: GND -> BLUE_LED_l
- U2 pad 3: VBAT_l -> (no net)
- U2 pad 4: VBUS_l -> /P0.28_l
- U2 pad 5: Net-(R2-Pad1) -> GND
- U3 pad 1: Net-(C3-Pad1) -> Net-(R8-Pad2)
- U3 pad 3: Net-(R1-Pad2) -> VBAT_l
- U3 pad 4: Net-(U3-Pad4) -> VBUS_l
- U3 pad 5: VCC -> Net-(R9-Pad1)
- U4 pad 1: Net-(U4-Pad1) -> Net-(D30-Pad1)
- U4 pad 3: Net-(U4-Pad3) -> Net-(D30-Pad1)
- U4 pad 4: DATA-_l -> (no net)
- U4 pad 5: Net-(F1-Pad2) -> nRF_VDD_r
- U5 pad 1: Net-(U5-Pad1) -> /P1.11_r
- U5 pad 2: GND -> BLUE_LED_r
- U5 pad 3: Net-(U5-Pad3) -> (no net)
- U5 pad 4: DATA-_r -> /P0.28_r
- U5 pad 5: Net-(F2-Pad2) -> GND
- U5 pad 6: DATA+_r -> /P1.13_r
- U6 pad 1: Net-(C4-Pad1) -> Net-(R17-Pad2)
- U6 pad 3: Net-(R13-Pad2) -> VBAT_r
- U6 pad 4: Net-(U6-Pad4) -> VBUS_r
- U6 pad 5: VCC -> Net-(R18-Pad1)
Other:
- board outline added: 326.2 x 104.8 mm

Commit message: Laaaazy...
Parts:
- added G3: LOGO, jiran-ble:logotype_rev, F.Cu at (155.2, 103.2)
- added G4: LOGO, jiran-ble:logotype_rev, F.Cu at (212.3, 106.0)
- moved G1 30.6 mm to (183.8, 90.9)
- moved G2 30.6 mm to (183.8, 90.9)
Routing:
- net /P0.29_l: track 0.00 -> 269.1 mm, vias 0 -> 1
- net /P0.29_r: track 0.00 -> 257.0 mm, vias 0 -> 1
- net GND: track 0.00 -> 222.4 mm, vias 0 -> 1
- net /P1.13_l: track 0.00 -> 211.2 mm, vias 0 -> 3
- net /P0.02_l: track 0.00 -> 211.0 mm, vias 0 -> 3
- net /P0.31_l: track 0.00 -> 205.6 mm, vias 0 -> 1
- net /P0.02_r: track 0.00 -> 203.3 mm, vias 0 -> 1
- net /P1.11_r: track 0.00 -> 202.6 mm, vias 0 -> 1
- net /P0.31_r: track 0.00 -> 197.5 mm, vias 0 -> 1
- net /P1.11_l: track 0.00 -> 192.1 mm, vias 0 -> 1
- net /P0.09_r: track 0.00 -> 183.6 mm, vias 0 -> 1
- net /P0.30_r: track 0.00 -> 175.1 mm, vias 0 -> 1
- net /P0.28_l: track 0.00 -> 174.5 mm, vias 0 -> 5
- net /P0.12_r: track 0.00 -> 174.1 mm
- net /P0.08_r: track 0.00 -> 173.5 mm, vias 0 -> 3
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- added copper zone on B.Cu, net (none)
- added copper zone on F.Cu, net (none)
Other:
- net class Default: clearance 0.2 -> 0.1; trace_width 0.25 -> 0.18; via_dia 0.8 -> 0.6; via_drill 0.4 -> 0.3
- rule trace_clearance: 0.2 -> 0.1
- rule trace_min: 0.2 -> 0.15
