File: pcb/jiran-ble/_autosave-jiran-ble.kicad_pcb (KiCad board)
At the start: 2 copper layers, 326.2 x 104.8 mm, 168 parts, among them J1 BATT, J2 USB-C Conn, J3 SWD, J4 BATT, J5 USB-C Conn, J6 SWD, P1 Breakoff, P2 Breakoff, P3 Breakoff, P4 Breakoff, Q1 AO3407, Q3 AO3407, SW1 SW_PUSH, SW10 SW_Push, SW11 SW_Push, SW12 SW_Push, SW13 SW_Push, SW14 SW_Push, SW15 SW_Push, SW16 SW_Push, SW17 SW_Push, SW18 SW_Push, SW19 SW_Push, SW2 SW_Push, SW20 SW_Push, SW21 SW_Push, SW22 SW_Push, SW23 SW_Push, SW24 SW_Push, SW25 SW_Push, SW26 SW_Push, SW27 SW_Push, SW28 SW_Push, SW29 SW_Push, SW3 SW_Push, SW30 SW_PUSH, SW31 SW_Push, SW32 SW_Push, SW33 SW_Push, SW34 SW_Push, SW35 SW_Push, SW36 SW_Push, SW37 SW_Push, SW38 SW_Push, SW39 SW_Push, SW4 SW_Push, SW40 SW_Push, SW41 SW_Push, SW42 SW_Push, SW43 SW_Push, SW44 SW_Push, SW45 SW_Push, SW46 SW_Push, SW47 SW_Push, SW48 SW_Push, SW49 SW_Push, SW5 SW_Push, SW50 SW_Push, SW51 SW_Push, SW52 SW_Push, SW53 SW_Push, SW54 SW_Push, SW55 SW_Push, SW56 SW_Push, SW57 SW_Push, SW58 SW_Push, SW6 SW_Push, SW7 SW_Push, SW8 SW_Push, SW9 SW_Push, U1 XC6220B331MR-G, U2 E73-2G4M08S1C, U3 TP4054, U4 XC6220B331MR-G, U5 E73-2G4M08S1C, U6 TP4054, X1 Crystal, X2 Crystal

Commit message: Laaaazy...
Parts:
- added G3: LOGO, jiran-ble:logotype_rev, F.Cu at (155.2, 103.2)
- added G4: LOGO, jiran-ble:logotype_rev, F.Cu at (212.3, 106.0)
Routing:
- net /P0.29_l: track 0.00 -> 269.1 mm, vias 0 -> 1
- net /P0.29_r: track 0.00 -> 257.0 mm, vias 0 -> 1
- net GND: track 0.00 -> 222.4 mm, vias 0 -> 1
- net /P1.13_l: track 0.00 -> 211.2 mm, vias 0 -> 3
- net /P0.02_l: track 0.00 -> 211.0 mm, vias 0 -> 3
- net /P0.31_l: track 0.00 -> 205.6 mm, vias 0 -> 1
- net /P0.02_r: track 0.00 -> 203.3 mm, vias 0 -> 1
- net /P1.11_r: track 0.00 -> 202.6 mm, vias 0 -> 1
- net /P0.31_r: track 0.00 -> 197.5 mm, vias 0 -> 1
- net /P1.11_l: track 0.00 -> 192.1 mm, vias 0 -> 1
- net /P0.09_r: track 0.00 -> 183.6 mm, vias 0 -> 1
- net /P0.30_r: track 0.00 -> 175.1 mm, vias 0 -> 1
- net /P0.28_l: track 0.00 -> 174.5 mm, vias 0 -> 5
- net /P0.12_r: track 0.00 -> 174.1 mm
- net /P0.08_r: track 0.00 -> 173.5 mm, vias 0 -> 3
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- added copper zone on B.Cu, net (none)
- added copper zone on F.Cu, net (none)
Other:
- net class Default: clearance 0.2 -> 0.1; trace_width 0.25 -> 0.18; via_dia 0.8 -> 0.6; via_drill 0.4 -> 0.3
- rule trace_clearance: 0.2 -> 0.1
- rule trace_min: 0.2 -> 0.15
