File: pcb/jiran-ble/jiran-ble.sch (KiCad schematic (older format))
At the start: 93 parts, among them J1 Conn_01x02, J2 Conn_01x04, J3 Conn_01x02, J4 Conn_01x02, Q1 AO3407, SW1 SW_Push, SW10 SW_Push, SW11 SW_Push, SW12 SW_Push, SW13 SW_Push, SW14 SW_Push, SW15 SW_Push, SW16 SW_Push, SW17 SW_Push, SW18 SW_Push, SW19 SW_Push, SW2 SW_Push, SW20 SW_Push, SW21 SW_Push, SW22 SW_Push, SW23 SW_Push, SW24 SW_Push, SW25 SW_Push, SW26 SW_Push, SW27 SW_Push, SW28 SW_Push, SW29 MSK-12C02, SW3 SW_Push, SW30 SW_PUSH, SW4 SW_Push, SW5 SW_Push, SW6 SW_Push, SW7 SW_Push, SW8 SW_Push, SW9 SW_Push, U1 E73-2G4M08S1C, U2 MCP73831, U3 AP2112K-3.3, U4 USBLC6-2SC6, Y1 Crystal

Commit message: Schematic is ready, create and add a lot of footprints
Parts:
- removed Y1: Crystal, Crystal:Crystal_SMD_3215-2Pin_3.2x1.5mm, symbol Device:Crystal
- C1, C2, C3: footprint Capacitor_SMD:C_0805_2012Metric -> jiran-ble:Capacitor_SMD_0805
- D1, D10, D11, D12, D13, D14, D15, D16, D17, D18, D19, D2, D20, D21, D22, D23, D24, D25, D26, D27, D28, D29, D3, D4, D5, D6, D7, D8, D9: footprint used_footprints:Diode_SMD_SOD-123 -> jiran-ble:Diode_SMD_SOD-123
- F1: footprint Fuse:Fuse_0805_2012Metric -> jiran-ble:Fuse_SMD_0805
- J1: footprint Connector_PinHeader_2.54mm:PinHeader_1x02_P2.54mm_Horizontal -> jiran-ble:Connector_THT_1x2_2.54
- J2: footprint Connector_PinHeader_2.54mm:PinHeader_1x04_P2.54mm_Vertical -> jiran-ble:Connector_THT_1x4_2.54
- J3, J4: footprint (none) -> jiran-ble:Connector_THT_1x2_2.54
- LED1, LED2: footprint LED_SMD:LED_0805_2012Metric -> jiran-ble:LED_SMD_0805
- Q1: footprint Package_TO_SOT_SMD:SOT-23 -> jiran-ble:Package_SMD_SOT-23
- R1, R2, R3, R4, R5, R6, R7, R8: footprint Resistor_SMD:R_0805_2012Metric -> jiran-ble:Resistor_SMD_0805
- SW1, SW10, SW11, SW12, SW13, SW14, SW15, SW16, SW17, SW18, SW19, SW2, SW20, SW21, SW22, SW23, SW24, SW25, SW26, SW27, SW28, SW3, SW4, SW5, SW6, SW7, SW8, SW9: footprint used_footprints:Switch_Mx_Hotswap_1u -> jiran-ble:Switch_Mx_Hotswap_1u
- SW29: footprint nrfmicro:switch_MSK-12C02_smd -> jiran-ble:Switch_SMD_MSK-12C02
- U1: footprint nrfmicro:E73-2G4M08S1C-52840 -> jiran-ble:E73-2G4M08S1C-52840
- U2, U3: footprint Package_TO_SOT_SMD:SOT-23-5 -> jiran-ble:Package_SMD_SOT-23-5
- U4: footprint Package_TO_SOT_SMD:SOT-23-6 -> jiran-ble:Package_SMD_SOT-23-6
- USB1: footprint nrfmicro:USB-C_C168688 -> jiran-ble:USB-C_MidMount
Connections:
- wire segments 161 -> 155
- no-connect marks 14 -> 16
Other:
- moved on the sheet: HC1, HC2, HM1, HM2, HM3, HM4, HM5, J2

Commit message: A lot of things, bruh
Parts:
- removed HC1, HC2: CoverHole, used_footprints:Hole_Cover_M2, symbol Mechanical:MountingHole
- added C4, C5: 10uF, jiran-ble:Capacitor_SMD_0805, symbol candy-rescue:C-nrfmicro-rescue
- added C6: 10uF, jiran-ble:Capacitor_SMD_0805, symbol Device:C
- added D30: 1N5819, jiran-ble:Diode_SMD_SOD-123, symbol candy-rescue:MBR0520-nrfmicro-rescue
- added D31, D32, D33, D34, D35, D36, D37, D38, D39, D40, D41, D42, D43, D44, D45, D46, D47, D48, D49, D50, D51, D52, D53, D54, D55, D56, D57, D58: 1N4148, jiran-ble:Diode_SMD_SOD-123, symbol Device:D_Small
- added F2: 500mA, jiran-ble:Fuse_SMD_0805, symbol Device:Polyfuse
- added HM10, HM6, HM7, HM8, HM9: CaseHole, used_footprints:Hole_Mount_M4, symbol Mechanical:MountingHole
- added J5, J7, J8: Conn_01x02, jiran-ble:Connector_THT_1x2_2.54, symbol Connector_Generic:Conn_01x02
- added J6: Conn_01x04, jiran-ble:Connector_THT_1x4_2.54, symbol Connector_Generic:Conn_01x04
- added LED3: BT, jiran-ble:LED_SMD_0805, symbol Device:LED
- added LED4: CHG, jiran-ble:LED_SMD_0805, symbol Device:LED
- added Q2: AO3407, jiran-ble:Package_SMD_SOT-23, symbol candy-rescue:BSS83P-nrfmicro-rescue
- added R10, R11: 5.1K, jiran-ble:Resistor_SMD_0805, symbol Device:R
- added R12, R15: 1K, jiran-ble:Resistor_SMD_0805, symbol Device:R
- added R13, R14: 100K, jiran-ble:Resistor_SMD_0805, symbol candy-rescue:R-nrfmicro-rescue
- added R16: 4.7K, jiran-ble:Resistor_SMD_0805, symbol Device:R
- added R9: 10K, jiran-ble:Resistor_SMD_0805, symbol candy-rescue:R-nrfmicro-rescue
- added SW31: SW_PUSH, jiran-ble:Switch_SMD_Tact_3-6-3,5, symbol candy-rescue:SW_PUSH-keyboard_parts
- added SW32: MSK-12C02, jiran-ble:Switch_SMD_MSK-12C02, symbol Switch:SW_SPDT
- added SW33, SW34, SW35, SW36, SW37, SW38, SW39, SW40, SW41, SW42, SW43, SW44, SW45, SW46, SW47, SW48, SW49, SW50, SW51, SW52, SW53, SW54, SW55, SW56, SW57, SW58, SW59, SW60: SW_Push, jiran-ble:Switch_Mx_Hotswap_1u, symbol Switch:SW_Push
- added U5: USBLC6-2SC6, jiran-ble:Package_SMD_SOT-23-6, symbol candy-rescue:USBLC6-2SC6-Power_Protection
- added U6: AP2112K-3.3, jiran-ble:Package_SMD_SOT-23-5, symbol candy-rescue:AP2112K-3.3-Regulator_Linear
- added U7: E73-2G4M08S1C, jiran-ble:E73-2G4M08S1C-52840, symbol candy-rescue:E73-2G4M08S1C-52840-nrfmicro
- added U8: MCP73831, jiran-ble:Package_SMD_SOT-23-5, symbol Battery_Management:MCP73831-2-OT
- added USB2: USB_C_Receptacle_USB2.0, jiran-ble:USB-C_MidMount, symbol candy-rescue:USB_C_Receptacle_USB2.0-Connector
- G1, G2: footprint used_footprints:Silk_Logo_Hotswap -> jiran-ble:logotype; symbol jiran:logo-jiran-hotswap -> jiran-ble:jiran-ble
- SW30: footprint Button_Switch_SMD:SW_DIP_SPSTx01_Slide_6.7x4.1mm_W6.73mm_P2.54mm_LowProfile_JPin -> jiran-ble:Switch_SMD_Tact_3-6-3,5
Connections:
- net labels added: BLUE_LED_l, BLUE_LED_r, BOOT_l, BOOT_r, DATA+_l, DATA+_r, DATA-_l, DATA-_r, DFU_l, DFU_r, P0.02_l, P0.02_r, P0.04_l, P0.04_r, P0.06_l, P0.06_r, P0.08_l, P0.08_r, P0.09_l, P0.09_r, P0.12_l, P0.12_r, P0.26_l, P0.26_r, P0.28_l, P0.28_r, P0.29_l, P0.29_r, P0.30_l, P0.30_r, P0.31_l, P0.31_r, P1.11_l, P1.11_r, P1.13_l, P1.13_r, RESET_l, RESET_r, SCL_l, SCL_r, SDA_l, SDA_r, SWC_l, SWC_r, SWD_l, SWD_r, SWO_l, SWO_r, VBAT_l, VBAT_r, VBUS_l, VBUS_r
- net labels removed: BLUE_LED, BOOT, DATA+, DATA-, DFU, P0.02, P0.04, P0.06, P0.08, P0.09, P0.12, P0.26, P0.28, P0.29, P0.30, P0.31, P1.11, P1.13, RESET, SCL, SDA, SWC, SWD, SWO, VBAT, VBUS
- wire segments 155 -> 318
- no-connect marks 16 -> 32
Other:
- note added: "31.01.21"
- note added: "Jiran-ble (left side) / r0.1 / 02.02.21"
- note added: "Jiran-ble (right side) / r0.1 / 02.02.21"
- note added: "Left side contain:\nSW1 - SW30\nD1 - D29\nR1 - R8\nHM1 - HM5\nU1 - U4\nJ1 - J4\nC1 - C3\nLED1 - LED2\nUSB1\nF1\nG1\n"
- note added: "Left side contain:\nSW31 - SW60\nD30 - D59\nR9 - R16\nHM6 - HM10\nU5 - U8\nJ5 - J8\nC4 - C6\nLED3 - LED4\nUSB2\nF2\nG2\n"
- note added: "Left side of PCB, be careful when making changes!"
- note added: "Right side of PCB, be careful when making changes!"
- note added: "jiran-ble"
- note added: "r0.1"
- note removed: "0.1"
- note removed: "31.01.2021"
- note removed: "Jiran-BLE"
- moved on the sheet: C1, C2, C3, D29, F1, J3, LED2, Q1, R1, R2, R3, R4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

Commit message: I am veeeery lazy...
Parts:
- removed C1, C3, C4, C5: 10uF, jiran-ble:Capacitor_SMD_0805, symbol candy-rescue:C-nrfmicro-rescue
- removed C2, C6: 10uF, jiran-ble:Capacitor_SMD_0805, symbol Device:C
- removed D29, D30: 1N5819, jiran-ble:Diode_SMD_SOD-123, symbol candy-rescue:MBR0520-nrfmicro-rescue
- removed F1, F2: 500mA, jiran-ble:Fuse_SMD_0805, symbol Device:Polyfuse
- removed J3, J5, J7, J8: Conn_01x02, jiran-ble:Connector_THT_1x2_2.54, symbol Connector_Generic:Conn_01x02
- removed Q1, Q2: AO3407, jiran-ble:Package_SMD_SOT-23, symbol candy-rescue:BSS83P-nrfmicro-rescue
- removed R1, R13, R14, R3: 100K, jiran-ble:Resistor_SMD_0805, symbol candy-rescue:R-nrfmicro-rescue
- removed R12, R15, R7: 1K, jiran-ble:Resistor_SMD_0805, symbol Device:R
- removed R16: 4.7K, jiran-ble:Resistor_SMD_0805, symbol Device:R
- removed R4, R5: 5.1K, jiran-ble:Resistor_SMD_0805, symbol Device:R
- removed R8, R9: 10K, jiran-ble:Resistor_SMD_0805, symbol candy-rescue:R-nrfmicro-rescue
- removed SW29, SW32: MSK-12C02, jiran-ble:Switch_SMD_MSK-12C02, symbol Switch:SW_SPDT
- removed SW31: SW_PUSH, jiran-ble:Switch_SMD_Tact_3-6-3,5, symbol candy-rescue:SW_PUSH-keyboard_parts
- removed SW59, SW60: SW_Push, jiran-ble:Switch_Mx_Hotswap_1u, symbol Switch:SW_Push
- removed U2, U8: MCP73831, jiran-ble:Package_SMD_SOT-23-5, symbol Battery_Management:MCP73831-2-OT
- removed U3, U6: AP2112K-3.3, jiran-ble:Package_SMD_SOT-23-5, symbol candy-rescue:AP2112K-3.3-Regulator_Linear
- removed U4, U5: USBLC6-2SC6, jiran-ble:Package_SMD_SOT-23-6, symbol candy-rescue:USBLC6-2SC6-Power_Protection
- removed U7: E73-2G4M08S1C, jiran-ble:E73-2G4M08S1C-52840, symbol candy-rescue:E73-2G4M08S1C-52840-nrfmicro
- removed USB1, USB2: USB_C_Receptacle_USB2.0, jiran-ble:USB-C_MidMount, symbol candy-rescue:USB_C_Receptacle_USB2.0-Connector
- added D1, D30: 1N5819, jiran-ble:Diode_SMD_SOD-123, symbol Device:D_Schottky_Small
- added J2, J5: USB-C Conn, jiran-ble:USB-C_MidMount, symbol nrfmicro-rescue:USB_C_Receptacle_USB2.0-Connector
- added Q1, Q3: AO3407, jiran-ble:Package_SMD_SOT-23, symbol Device:Q_PMOS_GSD
- added R1: 5.1K, jiran-ble:Resistor_SMD_0805, symbol Device:R
- added R12, R5: 820K, jiran-ble:Resistor_SMD_0805, symbol Device:R_Small
- added R13: 1K, jiran-ble:Resistor_SMD_0805, symbol Device:R
- added R15, R4: 100K, jiran-ble:Resistor_SMD_0805, symbol Device:R_Small
- added R16, R7: 2M, jiran-ble:Resistor_SMD_0805, symbol Device:R_Small
- added R17, R8: 1K, jiran-ble:Resistor_SMD_0805, symbol Device:R_Small
- added R18, R9: RPROG, jiran-ble:Resistor_SMD_0805, symbol Device:R_Small
- added SW30: SW_PUSH, jiran-ble:Switch_SMD_Tact_3-6-3,5, symbol candy-rescue:SW_PUSH-keyboard_parts
- added SW31, SW32: SW_Push, jiran-ble:Switch_Mx_Hotswap_1u, symbol Switch:SW_Push
- added U1, U4: XC6220B331MR-G, jiran-ble:Package_SMD_SOT-23-5, symbol nrfmicro-rescue:AP2112K-3.3-Regulator_Linear
- added U3, U6: TP4054, jiran-ble:Package_SMD_SOT-23-5, symbol Battery_Management:MCP73831-3-OT
- added U5: E73-2G4M08S1C, jiran-ble:E73-2G4M08S1C-52840, symbol candy-rescue:E73-2G4M08S1C-52840-nrfmicro
- added X1, X2: Crystal, jiran-ble:Crystal_SMD_CM9V, symbol Device:Crystal_Small
- HM1, HM10, HM2, HM3, HM4, HM5, HM6, HM7, HM8, HM9: footprint used_footprints:Hole_Mount_M4 -> jiran-ble:Hole_Mount_M4
- J1, J4: value Conn_01x02 -> BATT
- J3: renamed from J2; value Conn_01x04 -> SWD
- J6: value Conn_01x04 -> SWD
- LED2, LED4: value CHG -> RED
- R2: value 4.7K -> 5.1K
- renumbered D9 to D10, D10 to D11, D11 to D12, D12 to D13, D13 to D14, D14 to D15, D15 to D16, D16 to D17, D17 to D18, D18 to D19, D1 to D2, D19 to D20, D20 to D21, D21 to D22, D22 to D23, D23 to D24, D24 to D25, D25 to D26, D26 to D27, D27 to D28, D28 to D29, D2 to D3, D3 to D4, D4 to D5, D5 to D6, D6 to D7, D7 to D8, D8 to D9, R6 to R3, SW30 to SW1, SW9 to SW10, SW10 to SW11, SW11 to SW12, SW12 to SW13, SW13 to SW14, SW14 to SW15, SW15 to SW16, SW16 to SW17, SW17 to SW18, SW18 to SW19, SW1 to SW2, SW19 to SW20, SW20 to SW21, SW21 to SW22, SW22 to SW23, SW23 to SW24, SW24 to SW25, SW25 to SW26, SW26 to SW27, SW27 to SW28, SW28 to SW29, SW2 to SW3, SW3 to SW4, SW4 to SW5, SW5 to SW6, SW6 to SW7, SW7 to SW8, SW8 to SW9, U1 to U2
Connections:
- net BLUE_LED_r: now also U5.2 (P1.10)
- net DATA+_l: now also J2.A6 (D+), J2.B6 (D+)
- net DATA+_r: now also J5.A6 (D+), J5.B6 (D+), U5.31 (USB_D+)
- net DATA-_l: now also J2.A7 (D-), J2.B7 (D-)
- net DATA-_r: now also J5.A7 (D-), J5.B7 (D-), U5.29 (USB_D-)
- net GND: now also R10.2, R11.2, J2.A1 (GND), J2.A12 (GND), J2.B1 (GND), J2.B12 (GND), J2.S1 (SHIELD), J5.A1 (GND), J5.A12 (GND), J5.B1 (GND), J5.B12 (GND), J5.S1 (SHIELD), R1.2, R13.2, R15.2, R16.2, R18.2, R4.2, R7.2, R9.2, SW30.2, U1.2 (GND), U3.2 (VSS), U4.2 (GND), U5.21 (GND), U5.24 (GND), U5.5 (GND), U6.2 (VSS); no longer R10.1, R11.1
- net P0.02_r: now also U5.7 (P0.02/AIN0)
- net P0.06_r: now also SW33.2, SW39.2, SW45.2, SW51.2, U5.14 (P0.06); no longer SW35.2, SW41.2, SW47.2, SW53.2
- net P0.08_r: now also SW34.2, SW40.2, SW46.2, SW52.2, SW56.2, U5.16 (P0.08); no longer SW36.2, SW42.2, SW48.2, SW54.2, SW58.2
- net P0.09_r: now also SW35.2, SW41.2, SW47.2, SW53.2, SW57.2, U5.41 (P0.09/NFC1); no longer SW37.2, SW43.2, SW49.2, SW55.2
- net P0.12_r: now also SW36.2, SW42.2, SW48.2, SW54.2, SW58.2, U5.20 (P0.12); no longer SW38.2, SW44.2, SW50.2, SW56.2
- net P0.28_r: now also U5.4 (P0.28/AIN4)
- net P0.29_r: now also U5.8 (P0.29/AIN5)
- net P0.30_r: now also SW38.2, SW44.2, SW50.2, SW32.2, U5.10 (P0.30/AIN6); no longer SW34.2, SW40.2, SW46.2, SW52.2
- net P0.31_r: now also SW37.2, SW43.2, SW49.2, SW55.2, SW31.2, U5.9 (P0.31/AIN7); no longer SW33.2, SW39.2, SW45.2, SW51.2, SW57.2
- net P1.11_r: now also U5.1 (P1.11)
- net P1.13_r: now also U5.6 (P1.13)
- net RESET_r: now also SW30.1, U5.26 (P0.18/RESET)
- net SWC_r: now also U5.39 (SWDCLK)
- net SWD_r: now also U5.37 (SWDIO)
- net VBAT_l: now also Q1.3 (D), R5.1, U3.3 (VBAT)
- net VBAT_r: now also J4.2 (Pin_2), Q3.3 (D), R12.1, U6.3 (VBAT)
- net VBUS_l: now also D1.2 (A), J2.A4 (VBUS), J2.A9 (VBUS), J2.B4 (VBUS), J2.B9 (VBUS), Q1.1 (G), R4.1, U3.4 (VDD); no longer J4.2 (Pin_2)
- net VBUS_r: now also D30.2 (A), J5.A4 (VBUS), J5.A9 (VBUS), J5.B4 (VBUS), J5.B9 (VBUS), Q3.1 (G), R15.1, U5.27 (VBUS), U6.4 (VDD)
- net at R2.1: now also J2.B5 (CC2)
- net at U2.11 (P0.00/XL1): now also X1.1
- net at U2.13 (P0.01/XL2): now also X1.2
- net PROG_l: now reaches U2.15 (P0.05/AIN3)
- net POWER_PIN_l: now reaches U2.17 (P1.09)
- net nRF_VDD_l: now reaches U2.23 (VDDH)
- net nRF_VDD_l: now also J3.2 (Pin_2), U2.19 (VDD), U1.5 (VOUT)
- net DCCH_l: now reaches U2.25 (DCCH)
- net at LED2.1 (K): now also R8.1
- net at LED3.1 (K): now also R13.1
- net at LED4.1 (K): now also R17.1
- net at D31.2 (A): now also SW31.1; no longer SW33.1
- net at D32.2 (A): now also SW32.1; no longer SW34.1
- net at D33.2 (A): now also SW33.1; no longer SW35.1
- net at D34.2 (A): now also SW34.1; no longer SW36.1
- net at D35.2 (A): now also SW35.1; no longer SW37.1
- net at D36.2 (A): now also SW36.1; no longer SW38.1
- net at D37.2 (A): now also SW37.1; no longer SW39.1
- net at D38.2 (A): now also SW38.1; no longer SW40.1
- net at D39.2 (A): now also SW39.1; no longer SW41.1
- net at D40.2 (A): now also SW40.1; no longer SW42.1
- net at D41.2 (A): now also SW41.1; no longer SW43.1
- net at D42.2 (A): now also SW42.1; no longer SW44.1
- net at D43.2 (A): now also SW43.1; no longer SW45.1
- net at D44.2 (A): now also SW44.1; no longer SW46.1
- net at D45.2 (A): now also SW45.1; no longer SW47.1
- net at D46.2 (A): now also SW46.1; no longer SW48.1
- net at D47.2 (A): now also SW47.1; no longer SW49.1
- net at D48.2 (A): now also SW48.1; no longer SW50.1
- net at D49.2 (A): now also SW49.1; no longer SW51.1
- net at D50.2 (A): now also SW50.1; no longer SW52.1
- net at D51.2 (A): now also SW51.1; no longer SW53.1
- net at D52.2 (A): now also SW52.1; no longer SW54.1
- net at D53.2 (A): now also SW53.1; no longer SW55.1
- net at D54.2 (A): now also SW54.1; no longer SW56.1
- net at D55.2 (A): now also SW55.1; no longer SW57.1
- net at D56.2 (A): now also SW56.1; no longer SW58.1
- net at D57.2 (A): now also SW57.1
- net at D58.2 (A): now also SW58.1
- net BOOT_l: no longer names the net of U2.22 (P0.07)
- net DFU_l: no longer names the net of U2.38 (P1.02)
- net P0.04_l: no longer names the net of U2.12 (P0.26)
- net P0.04_l: no longer U2.18 (P0.04/AIN2)
- net SCL_l: no longer names the net of U2.30 (P0.17)
- net SDA_l: no longer names the net of U2.28 (P0.15)
- net SWO_l: no longer names the net of U2.36 (P1.00)
- removed net VCC: J3.2 (Pin_2), J6.2 (Pin_2), U2.19 (VDD)
- new net: D1.1 (K), Q1.2 (S), U1.1 (VIN), U1.3 (EN)
- new net: J2.A5 (CC1), R1.1
- new net: R8.2, U3.1 (STAT)
- new net: R9.1, U3.5 (PROG)
- new net: U5.11 (P0.00/XL1), X2.1
- new net: U5.13 (P0.01/XL2), X2.2
- new net: J5.B5 (CC2), R11.1
- new net: J5.A5 (CC1), R10.1
- new net: D30.1 (K), Q3.2 (S), U4.1 (VIN), U4.3 (EN)
- new net: R17.2, U6.1 (STAT)
- new net: R18.1, U6.5 (PROG)
- new net BATTERY_PIN_l: R5.2, R7.1, U2.18 (P0.04/AIN2)
- new net BATTERY_PIN_r: R12.2, R16.1, U5.18 (P0.04/AIN2)
- new net DCCH_r: U5.25 (DCCH)
- new net POWER_PIN_r: U5.17 (P1.09)
- new net PROG_r: U5.15 (P0.05/AIN3)
- new net nRF_VDD_r: J6.2 (Pin_2), U4.5 (VOUT), U5.19 (VDD), U5.23 (VDDH)
Other:
- note added: "Flags set \nonce for both halves!"
- note added: "IBat\n100mA\n200mA\n400mA\n500mA\n800mA"
- note added: "Jiran-ble (left side) / r0.2 / 06.02.21"
- note added: "Left side contain:\nSW1 - SW29\nD1 - D29\nR1 - R9\nHM1 - HM5\nU1 - U3\nJ1 - J3\nLED1 - LED2\nG1\n"
- note added: "Left side contain:\nSW30 - SW58\nD30 - D58\nR10 - R18\nHM6 - HM10\nU4 - U6\nJ4 - J6\nLED3 - LED4\nG2\n"
- note added: "LiPo Charging\n"
- note added: "Power Flags"
- note added: "RProg = 1000/IBat\nIBat in amps"
- note added: "RProg\n10k\n5k\n2.5k\n2k\n1.25k"
- note added: "r0.2"
- note removed: "Battery tester\n"
- note removed: "Jiran-ble (left side) / r0.1 / 02.02.21"
- note removed: "Jiran-ble (right side) / r0.1 / 02.02.21"
- note removed: "Left side contain:\nSW1 - SW30\nD1 - D29\nR1 - R8\nHM1 - HM5\nU1 - U4\nJ1 - J4\nC1 - C3\nLED1 - LED2\nUSB1\nF1\nG1\n"
- note removed: "Left side contain:\nSW31 - SW60\nD30 - D59\nR9 - R16\nHM6 - HM10\nU5 - U8\nJ5 - J8\nC4 - C6\nLED3 - LED4\nUSB2\nF2\nG2\n"
- note removed: "VBUS tester"
- note removed: "r0.1"
- moved on the sheet: J1, J3, LED1, R3, SW1

Commit message: Add power switch
Parts:
- added C?: 4.7uF, symbol Device:C_Small
- added SW?: SW_DPDT_x2, symbol Switch:SW_DPDT_x2
Connections:
- net GND: now also C?.2
- net VBAT_l: now also SW?.1 (A); no longer Q1.3 (D)
- net at D1.1 (K), Q1.2 (S), U1.1 (VIN)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: now also C?.1
- new net: Q1.3 (D), SW?.2 (B)
- no-connect marks 32 -> 33
Other:
- note removed: "Flags set \nonce for both halves!"
- moved on the sheet: Q1, R5, R7, U1
Changed lines of the file:
@@
 L Device:Q_PMOS_GSD Q1
 U 1 1 5B1587C5
-P 12225 2050
-F 0 "Q1" H 12425 2125 50  0000 L CNN
-F 1 "AO3407" H 12425 2050 50  0000 L CNN
-F 2 "jiran-ble:Package_SMD_SOT-23" H 12425 1975 50  0001 L CIN
-F 3 "" H 12225 2050 50  0001 L CNN
-	1    12225 2050
+P 12325 2050
+F 0 "Q1" H 12525 2125 50  0000 L CNN
+F 1 "AO3407" H 12525 2050 50  0000 L CNN
+F 2 "jiran-ble:Package_SMD_SOT-23" H 12525 1975 50  0001 L CIN
+F 3 "" H 12325 2050 50  0001 L CNN
+	1    12325 2050
 	1    0    0    -1
 $EndComp
 Text GLabel 11825 2050 0    60   Input ~ 0
 VBUS_l
-Wire Wire Line
-	13250 2400 13300 2400
 $Comp
 L nrfmicro-rescue:AP2112K-3.3-Regulator_Linear U1
 U 1 1 5EBF7400
-P 12950 2500
-F 0 "U1" H 12950 2842 50  0000 C CNN
-F 1 "XC6220B331MR-G" H 12950 2751 50  0000 C CNN
-F 2 "jiran-ble:Package_SMD_SOT-23-5" H 12950 2825 50  0001 C CNN
-F 3 "https://www.diodes.com/assets/Datasheets/AP2112.pdf" H 12950 2600 50  0001 C CNN
-	1    12950 2500
+P 12900 2500
+F 0 "U1" H 12900 2842 50  0000 C CNN
+F 1 "XC6220B331MR-G" H 12900 2751 50  0000 C CNN
+F 2 "jiran-ble:Package_SMD_SOT-23-5" H 12900 2825 50  0001 C CNN
+F 3 "https://www.diodes.com/assets/Datasheets/AP2112.pdf" H 12900 2600 50  0001 C CNN
+	1    12900 2500
 	1    0    0    -1
 $EndComp
@@
 	0    -1   1    0
 $EndComp
-Text GLabel 15000 2400 0    60   Input ~ 0
+Text GLabel 15525 2400 0    60   Input ~ 0
 BATTERY_PIN_l
-Text GLabel 15100 1950 1    60   Input ~ 0
+Text GLabel 15625 1950 1    60   Input ~ 0
 VBAT_l
 $Comp
 L Device:R_Small R7
 U 1 1 5ED6EA28
-P 15100 2625
-F 0 "R7" H 15170 2671 50  0000 L CNN
-F 1 "2M" H 15170 2580 50  0000 L CNN
-F 2 "jiran-ble:Resistor_SMD_0805" V 15030 2625 50  0001 C CNN
-F 3 "" H 15100 2625 50  0001 C CNN
-	1    15100 2625
+P 15625 2625
+F 0 "R7" H 15695 2671 50  0000 L CNN
+F 1 "2M" H 15695 2580 50  0000 L CNN
+F 2 "jiran-ble:Resistor_SMD_0805" V 15555 2625 50  0001 C CNN
+F 3 "" H 15625 2625 50  0001 C CNN
+	1    15625 2625
 	1    0    0    -1
 $EndComp
@@
 L Device:R_Small R5
 U 1 1 5ED6D985
-P 15100 2200
-F 0 "R5" H 15170 2246 50  0000 L CNN
-F 1 "820K" H 15170 2155 50  0000 L CNN
-F 2 "jiran-ble:Resistor_SMD_0805" V 15030 2200 50  0001 C CNN
-F 3 "" H 15100 2200 50  0001 C CNN
-	1    15100 2200
+P 15625 2200
+F 0 "R5" H 15695 2246 50  0000 L CNN
+F 1 "820K" H 15695 2155 50  0000 L CNN
+F 2 "jiran-ble:Resistor_SMD_0805" V 15555 2200 50  0001 C CNN
+F 3 "" H 15625 2200 50  0001 C CNN
+	1    15625 2200
 	1    0    0    -1
 $EndComp
@@
 $EndComp
 Wire Wire Line
-	15000 2400 15100 2400
-Connection ~ 15100 2400
-Wire Wire Line
-	12325 2250 12325 2400
-Text GLabel 12325 1750 1    60   Input ~ 0
+	15525 2400 15625 2400
+Connection ~ 15625 2400
+Text GLabel 12925 1650 2    60   Input ~ 0
 VBAT_l
 $Comp
@@
 	2775 4625 2875 4625
 $Comp
-L power:GND #PWR010
-U 1 1 5F7552D5
-P 12950 2800
-F 0 "#PWR010" H 12950 2550 50  0001 C CNN
-F 1 "GND" H 12950 2650 50  0000 C CNN
-F 2 "" H 12950 2800 50  0001 C CNN
-F 3 "" H 12950 2800 50  0001 C CNN
-	1    12950 2800
-	1    0    0    -1
-$EndComp
-$Comp
 L power:GND #PWR09
 U 1 1 5F7578BA
@@
 L power:GND #PWR018
 U 1 1 5F75E8D6
-P 15100 2725
-F 0 "#PWR018" H 15100 2475 50  0001 C CNN
-F 1 "GND" H 15100 2575 50  0000 C CNN
-F 2 "" H 15100 2725 50  0001 C CNN
-F 3 "" H 15100 2725 50  0001 C CNN
-	1    15100 2725
-	1    0    0    -1
-$EndComp
-Wire Wire Line
-	15100 2400 15100 2525
-Wire Wire Line
-	15100 2300 15100 2400
-Wire Wire Line
-	15100 1950 15100 2100
-Wire Wire Line
-	12550 2400 12650 2400
-Wire Wire Line
-	12650 2500 12550 2500
-Wire Wire Line
-	12550 2500 12550 2400
-Connection ~ 12550 2400
-Connection ~ 12325 2400
-Wire Wire Line
-	12325 2400 12550 2400
+P 15625 2725
+F 0 "#PWR018" H 15625 2475 50  0001 C CNN
+F 1 "GND" H 15625 2575 50  0000 C CNN
+F 2 "" H 15625 2725 50  0001 C CNN
+F 3 "" H 15625 2725 50  0001 C CNN
+	1    15625 2725
+	1    0    0    -1
+$EndComp
+Wire Wire Line
+	15625 2400 15625 2525
+Wire Wire Line
+	15625 2300 15625 2400
+Wire Wire Line
+	15625 1950 15625 2100
 $Comp
 L power:GND #PWR020
@@
 	1675 4625 1725 4625
 Wire Wire Line
-	12225 2400 12325 2400
-Wire Wire Line
 	11925 2500 11925 2400
 Wire Wire Line
@@
 	11925 2400 11925 2050
 Connection ~ 11925 2400
-Connection ~ 11925 2050
 Wire Wire Line
 	11825 2050 11925 2050
-Wire Wire Line
-	11925 2050 12025 2050
-Wire Wire Line
-	12325 1750 12325 1850
 NoConn ~ 5175 2200
 NoConn ~ 5175 2300
@@
 Wire Notes Line
 	11150 6425 11150 8650
-Text Notes 9700 6700 0    79   ~ 16
-Flags set \nonce for both halves!
+$Comp
+L Switch:SW_DPDT_x2 SW?
+U 1 1 6052BF4E
+P 12625 1750
+F 0 "SW?" H 12625 2035 50  0000 C CNN
+F 1 "SW_DPDT_x2" H 12625 1944 50  0000 C CNN
+F 2 "" H 12625 1750 50  0001 C CNN
+F 3 "~" H 12625 1750 50  0001 C CNN
+	1    12625 1750
+	1    0    0    -1
+$EndComp
+$Comp
+L Device:C_Small C?
+U 1 1 6052C804
+P 12325 2600
+F 0 "C?" H 12417 2646 50  0000 L CNN
+F 1 "4.7uF" H 12417 2555 50  0000 L CNN
+F 2 "" H 12325 2600 50  0001 C CNN
+F 3 "~" H 12325 2600 50  0001 C CNN
+	1    12325 2600
+	1    0    0    -1
+$EndComp
+Wire Wire Line
+	12225 2400 12325 2400
+Wire Wire Line
+	12325 2500 12325 2400
+Connection ~ 12325 2400
+Wire Wire Line
+	12325 2400 12425 2400
+Wire Wire Line
+	12425 2250 12425 2400
+Wire Wire Line
+	12125 2050 11925 2050
+Connection ~ 11925 2050
+Wire Wire Line
+	12925 1650 12825 1650
+Wire Wire Line
+	12425 1750 12425 1850
+NoConn ~ 12825 1850
+Wire Wire Line
+	12600 2400 12525 2400
+Connection ~ 12425 2400
+Wire Wire Line
+	12600 2500 12525 2500
+Wire Wire Line
+	12525 2500 12525 2400
+Connection ~ 12525 2400
+Wire Wire Line
+	12525 2400 12425 2400
+$Comp
+L power:GND #PWR010
+U 1 1 5F7552D5
+P 12900 2800
+F 0 "#PWR010" H 12900 2550 50  0001 C CNN
+F 1 "GND" H 12900 2650 50  0000 C CNN
+F 2 "" H 12900 2800 50  0001 C CNN
+F 3 "" H 12900 2800 50  0001 C CNN
+	1    12900 2800
+	1    0    0    -1
+$EndComp
+Wire Wire Line
+	13300 2400 13200 2400
+$Comp
+L power:GND #PWR0101
+U 1 1 605FE956
+P 12325 2700
+F 0 "#PWR0101" H 12325 2450 50  0001 C CNN
+F 1 "GND" H 12325 2550 50  0000 C CNN
+F 2 "" H 12325 2700 50  0001 C CNN
+F 3 "" H 12325 2700 50  0001 C CNN
+	1    12325 2700
+	1    0    0    -1
+$EndComp
+$Comp
+L power:PWR_FLAG #FLG0101
+U 1 1 60602024
+P 10075 7075
+F 0 "#FLG0101" H 10075 7150 50  0001 C CNN
+F 1 "PWR_FLAG" H 10075 7248 50  0000 C CNN
+F 2 "" H 10075 7075 50  0001 C CNN
+F 3 "~" H 10075 7075 50  0001 C CNN
+	1    10075 7075
+	0    -1   -1   0
+$EndComp
+Text GLabel 10075 7075 2    60   Input ~ 0
+nRF_VDD_r
+Text GLabel 10075 7975 2    60   Input ~ 0
+VBUS_r
+$Comp
+L power:PWR_FLAG #FLG0103
+U 1 1 60602038
+P 10075 7975
+F 0 "#FLG0103" H 10075 8050 50  0001 C CNN
+F 1 "PWR_FLAG" H 10075 8148 50  0000 C CNN
+F 2 "" H 10075 7975 50  0001 C CNN
+F 3 "~" H 10075 7975 50  0001 C CNN
+	1    10075 7975
+	0    -1   -1   0
+$EndComp
+Text GLabel 10075 7525 2    60   Input ~ 0
+VBAT_r
+$Comp
+L power:PWR_FLAG #FLG0104
+U 1 1 6060203F
+P 10075 7525
+F 0 "#FLG0104" H 10075 7600 50  0001 C CNN
+F 1 "PWR_FLAG" H 10075 7698 50  0000 C CNN
+F 2 "" H 10075 7525 50  0001 C CNN
+F 3 "~" H 10075 7525 50  0001 C CNN
+	1    10075 7525
+	0    -1   -1   0
+$EndComp
 $EndSCHEMATC
