File: pcb/jiran-ble/jiran-ble.sch (KiCad schematic (older format))
At the start: 166 parts, among them J1 BATT, J2 USB-C Conn, J3 SWD, J4 BATT, J5 USB-C Conn, J6 SWD, Q1 AO3407, Q3 AO3407, SW1 SW_PUSH, SW10 SW_Push, SW11 SW_Push, SW12 SW_Push, SW13 SW_Push, SW14 SW_Push, SW15 SW_Push, SW16 SW_Push, SW17 SW_Push, SW18 SW_Push, SW19 SW_Push, SW2 SW_Push, SW20 SW_Push, SW21 SW_Push, SW22 SW_Push, SW23 SW_Push, SW24 SW_Push, SW25 SW_Push, SW26 SW_Push, SW27 SW_Push, SW28 SW_Push, SW29 SW_Push, SW3 SW_Push, SW30 SW_PUSH, SW31 SW_Push, SW32 SW_Push, SW33 SW_Push, SW34 SW_Push, SW35 SW_Push, SW36 SW_Push, SW37 SW_Push, SW38 SW_Push, SW39 SW_Push, SW4 SW_Push, SW40 SW_Push, SW41 SW_Push, SW42 SW_Push, SW43 SW_Push, SW44 SW_Push, SW45 SW_Push, SW46 SW_Push, SW47 SW_Push, SW48 SW_Push, SW49 SW_Push, SW5 SW_Push, SW50 SW_Push, SW51 SW_Push, SW52 SW_Push, SW53 SW_Push, SW54 SW_Push, SW55 SW_Push, SW56 SW_Push, SW57 SW_Push, SW58 SW_Push, SW6 SW_Push, SW7 SW_Push, SW8 SW_Push, SW9 SW_Push, U1 XC6220B331MR-G, U3 TP4054, U4 XC6220B331MR-G, U5 E73-2G4M08S1C, U6 TP4054, X2 Crystal

Commit message: Remove some unused global net labels
Parts:
- removed Q3: AO3407, jiran-ble:Package_SMD_SOT-23, symbol Device:Q_PMOS_GSD
- removed R10, R11: 5.1K, jiran-ble:Resistor_SMD_0805, symbol Device:R
- removed R13: 1K, jiran-ble:Resistor_SMD_0805, symbol Device:R
- removed R17: 1K, jiran-ble:Resistor_SMD_0805, symbol Device:R_Small
- removed R18: RPROG, jiran-ble:Resistor_SMD_0805, symbol Device:R_Small
- removed SW30: SW_PUSH, jiran-ble:Switch_SMD_Tact_3-6-3,5, symbol candy-rescue:SW_PUSH-keyboard_parts
- removed SW31: SW_Push, jiran-ble:Switch_Mx_Hotswap_1u, symbol Switch:SW_Push
- removed U4: XC6220B331MR-G, jiran-ble:Package_SMD_SOT-23-5, symbol nrfmicro-rescue:AP2112K-3.3-Regulator_Linear
- removed U5: E73-2G4M08S1C, jiran-ble:E73-2G4M08S1C-52840, symbol candy-rescue:E73-2G4M08S1C-52840-nrfmicro
- removed X2: Crystal, jiran-ble:Crystal_SMD_CM9V, symbol Device:Crystal_Small
- added C3, C4: 4.7uF, symbol Device:C_Small
- added Q2: AO3407, jiran-ble:Package_SMD_SOT-23, symbol Device:Q_PMOS_GSD
- added R10, R9: 5.1k, symbol Device:R_Small
- added R11: 820K, jiran-ble:Resistor_SMD_0805, symbol Device:R_Small
- added R13: 100K, jiran-ble:Resistor_SMD_0805, symbol Device:R_Small
- added R14: 2M, jiran-ble:Resistor_SMD_0805, symbol Device:R_Small
- added unit 2 of SW2
- added SW31: SW_PUSH, jiran-ble:Switch_SMD_Tact_3-6-3,5, symbol candy-rescue:SW_PUSH-keyboard_parts
- added SW59: SW_Push, jiran-ble:Switch_Mx_Hotswap_1u, symbol Switch:SW_Push
- added U4: HOLYIOT-18010-NRF52840_simple, symbol jiran-ble:HOLYIOT-18010-NRF52840_simple
- added U5: XC6220B331MR-G, jiran-ble:Package_SMD_SOT-23-5, symbol nrfmicro-rescue:AP2112K-3.3-Regulator_Linear
- J2, J5: value USB-C Conn -> USB-C Connector
- R12: value 820K -> 1k; footprint jiran-ble:Resistor_SMD_0805 -> (none)
- R15: value 100K -> 1K
- R16: value 2M -> RPROG
- gave numbers to parts that had none: 7
- renumbered R5 to R3, R4 to R5, R7 to R6, R8 to R7, R9 to R8, SW9 to SW10, SW10 to SW11, SW11 to SW12, SW12 to SW13, SW13 to SW14, SW14 to SW15, SW15 to SW16, SW16 to SW17, SW17 to SW18, SW18 to SW19, SW19 to SW20, SW20 to SW21, SW21 to SW22, SW22 to SW23, SW23 to SW24, SW24 to SW25, SW25 to SW26, SW26 to SW27, SW27 to SW28, SW28 to SW29, SW2 to SW3, SW29 to SW30, SW3 to SW4, SW4 to SW5, SW5 to SW6, SW6 to SW7, SW7 to SW8, SW8 to SW9, U1 to U2
Connections:
- net labels added: D+_r, D-_r, P0.03_r, P0.19_r, P0.21_r, P0.23_r, P1.01_r, P1.03_r
- net labels removed: DATA+_l, DATA+_r, DATA-_l, DATA-_r, DCCH_r, P0.06_r, P0.08_r, P0.09_r, P0.12_r, P1.11_r, P1.13_r, POWER_PIN_l, POWER_PIN_r, PROG_l, PROG_r, SWO_l
- wire segments 251 -> 272
- no-connect marks 31 -> 36
Other:
- note added: "Jiran-ble (left side) / r0.3 / 18.03.21"
- note added: "Jiran-ble (right side) / r0.3 / 18.03.21"
- note added: "Left side contain:\nSW1 - SW30\nD1 - D29\nR1 - R9\nHM1 - HM5\nU1 - U3\nJ1 - J3\nLED1 - LED2\nC1 - C2\nG1\n"
- note added: "Right side contain:\nSW31 - SW59\nD30 - D58\nR10 - R18\nHM6 - HM10\nU4 - U6\nJ4 - J6\nLED3 - LED4\nC3 - C4\nG2\n"
- note added: "r0.3"
- note removed: "Jiran-ble (left side) / r0.2 / 06.02.21"
- note removed: "Left side contain:\nSW1 - SW29\nD1 - D29\nR1 - R9\nHM1 - HM5\nU1 - U3\nJ1 - J3\nLED1 - LED2\nG1\n"
- note removed: "Left side contain:\nSW30 - SW58\nD30 - D58\nR10 - R18\nHM6 - HM10\nU4 - U6\nJ4 - J6\nLED3 - LED4\nG2\n"
- note removed: "LiPo Charging\n"
- note removed: "USB"
- note removed: "r0.2"

Commit message: Fix a couple of errors
Connections:
- net SWD_L is gone; now on net SWD_l: U1.32 (SWDIO)
Other:
- note removed: "Power Flags"
- moved on the sheet: J1, J3, LED1, R4, SW1
